File: HARDWARE/Franzininho-Badge-2024/Franzininho-Badge-2024.kicad_pcb (KiCad board)
At the start: 2 copper layers, 96 x 64 mm, 68 parts, among them J1 UART, J2 SWIO, J3 SPI, Q1 SIL2308, SW1 USER, SW2 ON, SW3 RESET, U1 CH32V003F4P6, U2 OLED 128x64 1.3", U3 EPD 200x200 1.54"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

Commit message: Revisão de valores dos resistores. Geração de novo PDF do esquemático.
Parts:
- R10, R11, R12, R13, R14, R15, R16, R17, R6, R8: value 1K -> 47R
- R18, R19, R5: value 100K -> 10K
Changed lines of the file:
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@@
 		(grid_origin 139.7 101.6)
 		(pcbplotparams
-			(layerselection 0x00010f8_ffffffff)
+			(layerselection 0x00012a0_7ffffffe)
 			(plot_on_all_layers_selection 0x0000000_00000000)
 			(disableapertmacros no)
@@
 			(sketchpadsonfab no)
 			(subtractmaskfromsilk yes)
-			(outputformat 1)
+			(outputformat 4)
 			(mirror no)
 			(drillshape 0)
@@
 			)
 		)
-		(property "Value" "1K"
+		(property "Value" "47R"
 			(at 0 1.43 180)
 			(layer "F.Fab")
@@
 			)
 		)
-		(property "Value" "100K"
+		(property "Value" "10K"
 			(at 0 1.43 0)
 			(layer "F.Fab")
@@
 			)
 		)
-		(property "Value" "1K"
+		(property "Value" "47R"
 			(at 0 1.43 0)
 			(layer "F.Fab")
@@
 			)
 		)
-		(property "Value" "1K"
+		(property "Value" "47R"
 			(at 0 1.43 0)
 			(layer "F.Fab")
@@
 			)
 		)
-		(property "Value" "1K"
+		(property "Value" "47R"
 			(at 0 1.43 180)
 			(layer "F.Fab")
@@
 			)
 		)
-		(property "Value" "1K"
+		(property "Value" "47R"
 			(at 0 1.43 180)
 			(layer "F.Fab")
@@
 			)
 		)
-		(property "Value" "1K"
+		(property "Value" "47R"
 			(at 0 1.43 0)
 			(layer "F.Fab")
@@
 			)
 		)
-		(property "Value" "1K"
+		(property "Value" "47R"
 			(at 0 1.43 0)
 			(layer "F.Fab")
@@
 			)
 		)
-		(property "Value" "100K"
+		(property "Value" "10K"
 			(at 0 1.43 90)
 			(layer "F.Fab")
@@
 			)
 		)
-		(property "Value" "1K"
+		(property "Value" "47R"
 			(at 0 1.43 180)
 			(layer "F.Fab")
@@
 			)
 		)
-		(property "Value" "100K"
+		(property "Value" "10K"
 			(at 0 1.43 -90)
 			(layer "F.Fab")
@@
 			)
 		)
-		(property "Value" "1K"
+		(property "Value" "47R"
 			(at 0 1.43 180)
 			(layer "F.Fab")
@@
 			)
 		)
-		(property "Value" "1K"
+		(property "Value" "47R"
 			(at 0 1.43 180)
 			(layer "F.Fab")
